File: vco1_panel.brd (EAGLE design)
At the start: 128.5 x 50.5 mm, 4 parts

Commit message: Massive Changes, See Readme
Other:
- board text added: "D:/Text/Modular/TH-VCO1-master/Panel_Redesign_2/VCO1-Panel_Board-01.bmp"
- board text added: "Panel for Thomas Henry's VCO-1 Schematic adapted by Tom Witwell Design by David Huss Rev 1"
- board text removed: "Thomas Henry VCO1 Panel Designed by Tom Whitwell Herne Hill, London November 2015 PCB Rev 1"
