File: vco1_pots.sch (EAGLE design)
At the start: 27 parts

Commit message: Massive Changes, See Readme
Parts:
- added JP2, JP3: (no value), pinhead:PINHD-1X55X2MM
- 1V/OCT, EXP_FM, LINEAR_FM, PULSE_OUT, PWM_INPUT, SINE_OUT, TRIANGLE_OUT: value THONKICONNNEW -> WQP-PJ301M-12_JACK_LOW_SPACE; device MusicThingModular:THONKICONNNEW -> thonkiconn:WQP-PJ301M-12_JACK_LOW_SPACE
Connections:
- net GND: now also 1V/OCT.1, EXP_FM.1, JP2.1, JP2.2, JP2.3, JP2.4, JP2.5, JP3.1, JP3.2, JP3.3, JP3.4, JP3.5, LINEAR_FM.1, PULSE_OUT.1, PWM_INPUT.1, SINE_OUT.1, TRIANGLE_OUT.1; no longer 1V/OCT.SLEEVE, EXP_FM.SLEEVE, LINEAR_FM.SLEEVE, PULSE_OUT.SLEEVE, PWM_INPUT.SLEEVE, SINE_OUT.SLEEVE, TRIANGLE_OUT.SLEEVE
- net N$1: now also 1V/OCT.2; no longer 1V/OCT.TIP
- net N$18: now also TRIANGLE_OUT.2; no longer TRIANGLE_OUT.TIP
- net N$2: now also EXP_FM.2; no longer EXP_FM.TIP
- net N$20: now also LINEAR_FM.2; no longer LINEAR_FM.TIP
- net N$37: now also SINE_OUT.2; no longer SINE_OUT.TIP
- net N$41: now also PULSE_OUT.2; no longer PULSE_OUT.TIP
- net N$42: now also PWM_INPUT.2; no longer PWM_INPUT.TIP
