File: vco1_components.sch (EAGLE design)
At the start: 56 parts, among them IC1 LM13700N, Q3 2N3904, Q4 2N3904, U1 TL072_, U2 TL072_, U3 TL072_

Commit message: Massive Changes, See Readme
Parts:
- added JP2, JP3: (no value), pinhead:PINHD-1X55X2MM
- U$1: value THAT-340TRANSISTORS -> THAT-340; device MusicThingModular:THAT-340TRANSISTORS -> MusicThingModular:THAT-340THRUHOLE
Connections:
- net GND: now also JP2.1, JP2.2, JP2.3, JP2.4, JP2.5, JP3.1, JP3.2, JP3.3, JP3.4, JP3.5
Changed lines of the file:
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@@
 <?xml version="1.0" encoding="utf-8"?>
 <!DOCTYPE eagle SYSTEM "eagle.dtd">
-<eagle version="7.2.0">
+<eagle version="7.6.0">
 <drawing>
 <settings>
@@
 <layer number="2" name="Route2" color="1" fill="3" visible="no" active="no"/>
 <layer number="3" name="Route3" color="4" fill="3" visible="no" active="no"/>
+<layer number="4" name="Route4" color="1" fill="4" visible="no" active="no"/>
+<layer number="5" name="Route5" color="4" fill="4" visible="no" active="no"/>
+<layer number="6" name="Route6" color="1" fill="8" visible="no" active="no"/>
+<layer number="7" name="Route7" color="4" fill="8" visible="no" active="no"/>
+<layer number="8" name="Route8" color="1" fill="2" visible="no" active="no"/>
+<layer number="9" name="Route9" color="4" fill="2" visible="no" active="no"/>
+<layer number="10" name="Route10" color="1" fill="7" visible="no" active="no"/>
+<layer number="11" name="Route11" color="4" fill="7" visible="no" active="no"/>
+<layer number="12" name="Route12" color="1" fill="5" visible="no" active="no"/>
+<layer number="13" name="Route13" color="4" fill="5" visible="no" active="no"/>
 <layer number="14" name="Route14" color="1" fill="6" visible="no" active="no"/>
 <layer number="15" name="Route15" color="4" fill="6" visible="no" active="no"/>
@@
 <part name="SUPPLY38" library="supply2" deviceset="GND" device=""/>
 <part name="R36" library="MusicThingModular" deviceset="RESISTOR" device="7MM" value="150k"/>
-<part name="U$1" library="MusicThingModular" deviceset="THAT-340" device="TRANSISTORS"/>
+<part name="U$1" library="MusicThingModular" deviceset="THAT-340" device="THRUHOLE" value="THAT-340"/>
 <part name="SV1" library="MusicThingModular" deviceset="EURO_POWER_HEADER" device="LOCK_PADS"/>
 <part name="SUPPLY39" library="supply2" deviceset="-12V" device=""/>
@@
 <part name="C14" library="TomW" deviceset="C-EU" device="050-024X044" value="100n"/>
 <part name="JP1" library="SparkFun-Connectors" deviceset="M10" device="&quot;"/>
+<part name="SUPPLY1" library="supply2" deviceset="GND" device=""/>
+<part name="JP2" library="pinhead" deviceset="PINHD-1X5" device="5X2MM"/>
+<part name="SUPPLY2" library="supply2" deviceset="GND" device=""/>
+<part name="JP3" library="pinhead" deviceset="PINHD-1X5" device="5X2MM"/>
 </parts>
 <sheets>
@@
 <instance part="C14" gate="G$1" x="426.72" y="111.76"/>
 <instance part="JP1" gate="G$1" x="396.24" y="220.98"/>
+<instance part="SUPPLY1" gate="GND" x="370.84" y="200.66"/>
+<instance part="JP2" gate="A" x="360.68" y="210.82" rot="R180"/>
+<instance part="SUPPLY2" gate="GND" x="370.84" y="226.06"/>
+<instance part="JP3" gate="A" x="360.68" y="236.22" rot="R180"/>
 </instances>
 <busses>
@@
 <segment>
 <pinref part="JP1" gate="G$1" pin="9"/>
-<wire x1="408.94" y1="223.52" x2="406.4" y2="223.52" width="0.1524" layer="91"/>
-<label x="408.94" y="223.52" size="1.4224" layer="95" xref="yes"/>
+<wire x1="406.4" y1="223.52" x2="408.94" y2="223.52" width="0.1524" layer="91"/>
+<label x="408.94" y="223.52" size="1.27" layer="95" xref="yes"/>
+</segment>
+<segment>
+<pinref part="JP2" gate="A" pin="5"/>
+<wire x1="363.22" y1="215.9" x2="370.84" y2="215.9" width="0.1524" layer="91"/>
+<wire x1="370.84" y1="215.9" x2="370.84" y2="213.36" width="0.1524" layer="91"/>
+<pinref part="JP2" gate="A" pin="4"/>
+<wire x1="370.84" y1="213.36" x2="363.22" y2="213.36" width="0.1524" layer="91"/>
+<pinref part="JP2" gate="A" pin="3"/>
+<wire x1="370.84" y1="213.36" x2="370.84" y2="210.82" width="0.1524" layer="91"/>
+<wire x1="370.84" y1="210.82" x2="363.22" y2="210.82" width="0.1524" layer="91"/>
+<junction x="370.84" y="213.36"/>
+<pinref part="JP2" gate="A" pin="2"/>
+<wire x1="370.84" y1="210.82" x2="370.84" y2="208.28" width="0.1524" layer="91"/>
+<wire x1="370.84" y1="208.28" x2="363.22" y2="208.28" width="0.1524" layer="91"/>
+<junction x="370.84" y="210.82"/>
+<pinref part="JP2" gate="A" pin="1"/>
+<wire x1="370.84" y1="208.28" x2="370.84" y2="205.74" width="0.1524" layer="91"/>
+<wire x1="370.84" y1="205.74" x2="363.22" y2="205.74" width="0.1524" layer="91"/>
+<junction x="370.84" y="208.28"/>
+<pinref part="SUPPLY1" gate="GND" pin="GND"/>
+<wire x1="370.84" y1="205.74" x2="370.84" y2="203.2" width="0.1524" layer="91"/>
+<junction x="370.84" y="205.74"/>
+</segment>
+<segment>
+<pinref part="JP3" gate="A" pin="5"/>
+<wire x1="363.22" y1="241.3" x2="370.84" y2="241.3" width="0.1524" layer="91"/>
+<wire x1="370.84" y1="241.3" x2="370.84" y2="238.76" width="0.1524" layer="91"/>
+<pinref part="JP3" gate="A" pin="4"/>
+<wire x1="370.84" y1="238.76" x2="363.22" y2="238.76" width="0.1524" layer="91"/>
+<pinref part="JP3" gate="A" pin="3"/>
+<wire x1="370.84" y1="238.76" x2="370.84" y2="236.22" width="0.1524" layer="91"/>
+<wire x1="370.84" y1="236.22" x2="363.22" y2="236.22" width="0.1524" layer="91"/>
+<junction x="370.84" y="238.76"/>
+<pinref part="JP3" gate="A" pin="2"/>
+<wire x1="370.84" y1="236.22" x2="370.84" y2="233.68" width="0.1524" layer="91"/>
+<wire x1="370.84" y1="233.68" x2="363.22" y2="233.68" width="0.1524" layer="91"/>
+<junction x="370.84" y="236.22"/>
+<pinref part="JP3" gate="A" pin="1"/>
+<wire x1="370.84" y1="233.68" x2="370.84" y2="231.14" width="0.1524" layer="91"/>
+<wire x1="370.84" y1="231.14" x2="363.22" y2="231.14" width="0.1524" layer="91"/>
+<junction x="370.84" y="233.68"/>
+<pinref part="SUPPLY2" gate="GND" pin="GND"/>
+<wire x1="370.84" y1="231.14" x2="370.84" y2="228.6" width="0.1524" layer="91"/>
+<junction x="370.84" y="231.14"/>
 </segment>
 </net>

Commit message: Cleanup of the Board schematics
Other:
- note added: "Discrete Schmitt Trigger"
- note added: "Exponential Converter"
- note added: "Opamp Integrator"
- note added: "Oscillator Core (Schmitt Trigger Integrator)"
- note added: "PWM Comparator"
- note added: "Power Section & Connectors"
- note added: "Sine Waveshaper"
- note added: "Unused LM13700 Pins"
- moved on the sheet: C1, C10, C11, C12, C13, C14, C3, C4, C5, C6, C7, C8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
